File: ProtectionCircuit.kicad_sch (KiCad schematic)
At the start: 22 parts, among them SW2 SW_DIP_x01, SW3 SW_DIP_x01

Commit message: Final Schematic
Final Schematic. PC104 pins not assigned.
Parts:
- removed SW2, SW3: SW_DIP_x01, Button_Switch_SMD:SW_DIP_SPSTx01_Slide_6.7x4.1mm_W6.73mm_P2.54mm_LowProfile_JPin, symbol Switch:SW_DIP_x01
- added C42, C46, C62: 10uF, fp:CAPC2012X94N, symbol 0805YC106KAT2A:0805YC106KAT2A
- added C43, C47, C63: 100pF, fp:CAPC1005X55N, symbol C0402C101K3RACAUTO:C0402C101K3RACAUTO
- added C44, C48, C64: 100nF, fp:C1005_Commercial, symbol C1005X7R1C104K050BC:C1005X7R1C104K050BC
- added C45, C49, C65: 1uF, fp:C2220_FT, symbol C2220X105K2RACAUTO:C2220X105K2RACAUTO
- added F3, F4, F6: TPS25961DRVR, fp:SON65P200X200X80-7N, symbol TPS25961DRVR:TPS25961DRVR
- added Q1, Q2, Q3, Q4, Q5: NPN, symbol Simulation_SPICE:NPN
- added R38: 100k, fp:RC0603FR-072ML, symbol 2023-02-18_05-38-06:RC0603FR-072ML
- added R39, R42, R44, R47, R62, R65: 2M, fp:RC0603FR-072ML, symbol 2023-02-18_05-38-06:RC0603FR-072ML
- added R40: 953k, fp:RC0603FR-072ML, symbol 2023-02-18_05-38-06:RC0603FR-072ML
- added R41: 1.54M, fp:RC0603FR-072ML, symbol 2023-02-18_05-38-06:RC0603FR-072ML
- added R43, R61: 50.5k, fp:RC0603FR-072ML, symbol 2023-02-18_05-38-06:RC0603FR-072ML
- added R45, R63: 549k, fp:RC0603FR-072ML, symbol 2023-02-18_05-38-06:RC0603FR-072ML
- added R46, R64: 787k, fp:RC0603FR-072ML, symbol 2023-02-18_05-38-06:RC0603FR-072ML
- added R? (x5): 50m, symbol Device:R_Small
Connections:
- net Earth: now also C42.2, C43.2, C44.2, C45.2, C46.2, C47.2, C48.2, C49.2, C62.2, C63.2, C64.2, C65.2, F3.4 (GND_1), F3.7 (GND_2), F4.4 (GND_1), F4.7 (GND_2), F6.4 (GND_1), F6.7 (GND_2), Q1.3 (E), Q2.3 (E), Q3.3 (E), Q4.3 (E), Q5.3 (E), R38.2, R40.2, R41.2, R43.2, R45.2, R46.2, R61.2, R63.2, R64.2
- net at C23.1, F1.5 (EN/UVLO), R17.1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: now also Q1.1 (C)
- net at C27.1, F2.5 (EN/UVLO), R22.1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: now also Q3.1 (C)
- net 3.3Vin renamed 3.3V_COMM
- net 3.3Vout renamed 3.3Vout_COMM
- net 5Vin renamed 5V_OBC
- net 5Vout renamed 5Vout_OBC
- new net: C43.1, F3.5 (EN/UVLO), Q2.1 (C), R41.1, R42.2
- new net: Q2.2 (B), R?.1
- new net: F4.2 (OVLO), R44.2, R45.1
- new net: F6.3 (ILIM), R61.1
- new net: C47.1, F4.5 (EN/UVLO), Q4.1 (C), R46.1, R47.2
- new net: Q3.2 (B), R?.1
- new net: C63.1, F6.5 (EN/UVLO), Q5.1 (C), R64.1, R65.2
- new net: F3.3 (ILIM), R38.1
- new net: Q1.2 (B), R?.1
- new net: F3.2 (OVLO), R39.2, R40.1
- new net: F6.2 (OVLO), R62.2, R63.1
- new net: F4.3 (ILIM), R43.1
- new net: Q5.2 (B), R?.1
- new net: Q4.2 (B), R?.1
- new net 3.3V_ADCS: C44.1, C45.1, F3.6 (IN), R39.1, R42.1
- new net 3.3V_ADCS_EN: R?.2
- new net 3.3V_COMM_EN: R?.2
- new net 3.3Vout_ADCS: C42.1, F3.1 (OUT)
- new net 5V_COMM: C64.1, C65.1, F6.6 (IN), R62.1, R65.1
- new net 5V_COMM_EN: R?.2
- new net 5V_OBC_EN: R?.2
- new net 5V_PAYLOAD: C48.1, C49.1, F4.6 (IN), R44.1, R47.1
- new net 5V_PAYLOAD_EN: R?.2
- new net 5Vout_COMM: C62.1, F6.1 (OUT)
- new net 5Vout_PAYLOAD: C46.1, F4.1 (OUT)
Other:
- moved on the sheet: C22, C23, C24, C25, C26, C27, C28, C29, F1, F2, R14, R15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

Commit message: Ready to rearrange
Parts:
- C22, C26, C42, C46, C62: footprint fp:CAPC2012X94N -> 10uF MLCC:CAPC2012X94N
- C23, C27, C43, C47, C63: footprint fp:CAPC1005X55N -> 10uF MLCC:CAPC2012X94N
- C24, C28, C44, C48, C64: footprint fp:C1005_Commercial -> 10uF MLCC:CAPC2012X94N
- C25, C29, C45, C49, C65: footprint fp:C2220_FT -> 10uF MLCC:CAPC2012X94N
- F1, F2, F3, F4, F6: footprint fp:SON65P200X200X80-7N -> PROTECC:SON65P200X200X80-7N
- Q1, Q2, Q3, Q4, Q5: footprint (none) -> bjt:PBSS4310PASQX
- R14, R15, R16, R17, R18, R19, R20, R21, R22, R23, R38, R39, R40, R41, R42, R43, R44, R45, R46, R47, R61, R62, R63, R64, R65: footprint fp:RC0603FR-072ML -> Resistor_SMD:R_0805_2012Metric
- R? (x5): footprint (none) -> Resistor_SMD:R_0805_2012Metric

Commit message: updates
Other:
- moved on the sheet: C22, C23, C24, C25, C26, C27, C28, C29, C42, C43, C44, C45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
