File: pcb.kicad_pcb (KiCad board)
At the start: 4 copper layers, 95.1 x 95.1 mm, 186 parts, among them IC1 BQ25302RTER, IC2 SPV1040T, IC3 SI3483DDV-T1-BE3, IC4 SPV1040T, IC5 SPV1040T, J1 PTHF-126-02-GF-Q-368, J2 Sol_X+_X-, J3 Sol_Y+_Y-, J4 USB_B_Micro, J5 SWD, J6 Sol_Z+_Z-, Q1 NPN, Q2 NPN, Q3 NPN, Q4 NPN, Q5 NPN, SW1 SW_SPDT, U1 STM32F405RGT6, U2 LTC2990, U3 LTC2990, U4 LTC2990, Y1 16MHz

Commit message: Arranged
Parts:
- SW1: moved to B.Cu
- moved C49 180.8 mm to (271.8, 130.3)
- moved C62 180.8 mm to (271.8, 133.2)
- moved C63 180.8 mm to (271.8, 136.0)
- moved C64 180.8 mm to (271.8, 138.8)
- moved C65 180.8 mm to (271.8, 141.7)
- moved C27 180.8 mm to (263.8, 130.3)
- moved C28 180.8 mm to (263.8, 133.2)
- moved C29 180.8 mm to (263.8, 136.0)
- moved C42 180.8 mm to (263.8, 138.8)
- moved C43 180.8 mm to (263.8, 141.7)
- moved C44 180.8 mm to (267.8, 130.3)
- moved C45 180.8 mm to (267.8, 133.2)
- moved C46 180.8 mm to (267.8, 136.0)
- moved C47 180.8 mm to (267.8, 138.8)
- moved C48 180.8 mm to (267.8, 141.7)
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Routing:
- added copper zone on F.Cu, net +Vpp
- removed copper zone on In2.Cu, net 5V

Commit message: LIBS + 3D EXPORT, Ready to reroute
Parts:
- BT1: footprint Battery:BatteryHolder_Keystone_1042_1x18650 -> Library:BatteryHolder_Keystone_1042_1x18650
- Boost_IC1, Boost_IC2, Boost_IC3: footprint Boost LTC3426:SOT95P280X90-6N -> Library:SOT95P280X90-6N
- Buck_IC1, Buck_IC2, Buck_IC3: footprint BUck TPS62203DBVT:SOT95P280X145-5N -> Library:SOT95P280X145-5N
- C1, C50, C54: footprint cap 4.7uf:C1210 -> Library:C1210
- C10, C14, C16: footprint Capacitor_SMD:C_0603_1608Metric -> Library:C_0603_1608Metric
- C11, C12, C13, C15, C17, C18, C19, C20, C21: footprint Capacitor_SMD:C_0402_1005Metric -> Library:C_0402_1005Metric
- C2, C22, C23, C24, C25, C26, C27, C28, C29, C3, C30, C33, C34, C36, C38, C40, C42, C43, C44, C45, C46, C47, C48, C49, C51, C52, C55, C56, C6, C62, C63, C64, C65, C8: footprint 10uF MLCC:CAPC2012X94N -> Library:CAPC2012X94N
- C31, C5: footprint 2.2uF:CAPC0603X33N -> Library:CAPC0603X33N
- C32, C35, C37, C39, C41, C7, C9: footprint 47nF:C1005_Commercial -> Library:C1005_Commercial
- C4, C53, C57: footprint cap 22uF low esr and esl:C3216_Commercial -> Library:C3216_Commercial
- D1, D10, D11, D12, D13, D14, D2, D4, D5, D6, D7, D8, D9: footprint Schottky DD with stock:DIOM5126X265N -> Library:DIOM5126X265N
- D3: footprint LED_SMD:LED_0603_1608Metric -> Library:LED_0603_1608Metric
- F1, F2, F3, F4, F6: footprint PROTECC:SON65P200X200X80-7N -> Library:SON65P200X200X80-7N
- IC1: footprint Charger bq 25302:QFN50P300X300X80-17N-D -> Library:QFN50P300X300X80-17N-D
- IC2, IC4, IC5: footprint MPPT:SPV1040T -> Library:SPV1040T
- IC3: footprint PFET:SOT95P284X110-6N -> Library:SOT95P284X110-6N
- J1: footprint CONN PC104:CONN_PTHF-126-02-GF-Q-368_SAI -> Library:CONN_PTHF-126-02-GF-Q-368_SAI
- J2, J3, J6: footprint Connector_JST:JST_GH_SM04B-GHS-TB_1x04-1MP_P1.25mm_Horizontal -> Library:JST_GH_SM04B-GHS-TB_1x04-1MP_P1.25mm_Horizontal
- J4: footprint usbb:USB_Micro-B_Amphenol_10118194_Horizontal -> Library:USB_Micro-B_Amphenol_10118194_Horizontal
- J5: footprint Connector_PinHeader_1.00mm:PinHeader_2x05_P1.00mm_Vertical_SMD -> Library:PinHeader_2x05_P1.00mm_Vertical_SMD
- L1, L10, L8: footprint indc 2.2uH:IHLP2020CZER2R2M8A -> Library:IHHP0805ZHER1R0M01
- L11, L2, L4, L6, L7, L9: footprint indc 10uH crct:SRN1060-100M -> Library:IHLP2020CZER2R2M8A
- L3: footprint Inductor_SMD:L_0402_1005Metric -> Library:L_0402_1005Metric
- L5: footprint 1uH indc:IHHP0805ZHER1R0M01 -> Library:IHHP0805ZHER1R0M01
- Q1, Q2, Q3, Q4, Q5: footprint bjt:PBSS4310PASQX -> Library:PBSS4310PASQX
- R10, R11, R12, R13: footprint Resistor_SMD:R_0402_1005Metric -> Library:R_0402_1005Metric
- R14, R15, R16, R17, R18, R19, R20, R21, R22, R23, R26, R27, R28, R29, R30, R31, R32, R33, R34, R35, R36, R37, R38, R39, R40, R41, R42, R43, R44, R45, R46, R47, R56, R57, R58, R6, R61, R62, R63, R64, R65, R66, R67, R68, R69, R7, R70, R8: footprint Resistor_SMD:R_0805_2012Metric -> Library:R_0805_2012Metric
- R2, R49, R53: footprint 1MEGA RST:RESC1608X55N -> Library:RESC1608X55N
- R24, R25, R4, R5, R51, R55: footprint rst 30.9k:RC0603FR-0730K9L -> Library:RC0603FR-0730K9L
- R3, R50, R54: footprint rst 95.3k:RESC2012X60N -> Library:RESC2012X60N
- R9: footprint Resistor_SMD:R_0603_1608Metric -> Library:R_0603_1608Metric
- SW1: footprint Button_Switch_SMD:SW_SPDT_PCM12 -> Library:SW_SPDT_PCM12
- TH1: footprint Thermmy:103AT2 -> Library:103AT2
- U1: footprint Package_QFP:LQFP-64_10x10mm_P0.5mm -> Library:LQFP-64_10x10mm_P0.5mm
- U2, U3, U4: footprint MON & PROTECC:SOP50P490X110-10N -> Library:SOP50P490X110-10N
- Y1: footprint Crystal:Crystal_SMD_3225-4Pin_3.2x2.5mm -> Library:Crystal_SMD_3225-4Pin_3.2x2.5mm
- moved R20 101.1 mm to (141.6, 109.0), turned to 90 degrees
- moved R40 97.6 mm to (141.6, 104.6), turned to 90 degrees
- moved R21 95.7 mm to (146.6, 109.1), turned to 90 degrees
- moved R46 94.4 mm to (141.6, 100.2), turned to 90 degrees
- moved R41 92.1 mm to (146.6, 104.6), turned to 90 degrees
- moved L5 91.6 mm to (171.6, 87.3)
- moved IC2 91.6 mm to (122.4, 60.0)
- moved J1 91.6 mm to (119.0, 32.6)
- moved Boost_IC2 91.6 mm to (154.8, 67.1)
- moved C49 91.6 mm to (183.3, 106.5)
- moved C64 91.6 mm to (183.3, 115.0)
- moved R12 91.6 mm to (177.5, 69.7)
- moved R13 91.6 mm to (179.5, 69.7)
- moved R7 91.6 mm to (103.6, 87.5)
- moved C36 91.6 mm to (113.5, 84.0)
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Routing:
- removed copper zone on In1.Cu, net +3.3V
Other:
- copper layers 4 -> 2

Commit message: updates
Routing:
- net Earth: track 0.00 -> 628.9 mm, vias 0 -> 1
- net +Vpp: track 0.00 -> 182.2 mm, vias 0 -> 16
- net 3.3V_ADCS: track 0.00 -> 156.9 mm, vias 0 -> 4
- net 5V_PAYLOAD: track 0.00 -> 134.7 mm, vias 0 -> 2
- net +3V3: track 0.00 -> 110.3 mm, vias 0 -> 1
- net MPPT_I+: track 0.00 -> 105.4 mm
- net GND: track 0.00 -> 93.8 mm, vias 0 -> 8
- net BAT_I-: track 0.00 -> 83.3 mm, vias 0 -> 2
- net SOL_Y_ADC: track 0.00 -> 77.4 mm, vias 0 -> 2
- net Net-(IC1-TS): track 0.00 -> 77.0 mm, vias 0 -> 1
- net Net-(D11-K): track 0.00 -> 76.9 mm, vias 0 -> 2
- net 5V_COMM: track 0.00 -> 76.0 mm
- net Net-(IC5-VCTRL): track 0.00 -> 73.6 mm, vias 0 -> 3
- net MPPT_I-: track 0.00 -> 63.3 mm, vias 0 -> 3
- net 3.3V_COMM: track 0.00 -> 59.7 mm
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Other:
- copper layers 2 -> 4
