File: pcb.kicad_sch (KiCad schematic)
At the start: 1 part, among them J1 PTHF-126-02-GF-Q-368

Commit message: Ready to rearrange
Connections:
- net +3.3V: now reaches J1.1
- net +3.3V: now also J1.2
- net 3.3V_COMM: now reaches J1.10
- net 3.3V_COMM: now also J1.9
- net 5V: now reaches J1.3
- net 5V: now also J1.4
- net 3.3V_ADCS: now reaches J1.5
- net 3.3V_ADCS: now also J1.6
- net 5V_PAYLOAD: now reaches J1.7
- net 5V_PAYLOAD: now also J1.8
Other:
- moved on the sheet: J1A, J1B, J1C
Changed lines of the file:
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@@
 (kicad_sch (version 20230121) (generator eeschema)
   (paper "A4")
-  (symbol (lib_id "PC104 conn:PTHF-126-02-GF-Q-368") (at 227.33 54.61 0) (unit 1)
+  (junction (at 270.51 71.12) (diameter 0) (color 0 0 0 0)
+  )
+  (junction (at 270.51 55.88) (diameter 0) (color 0 0 0 0)
+  )
+  (junction (at 270.51 66.04) (diameter 0) (color 0 0 0 0)
+  )
+  (junction (at 270.51 76.2) (diameter 0) (color 0 0 0 0)
+  )
+  (junction (at 270.51 60.96) (diameter 0) (color 0 0 0 0)
+  )
+  (wire (pts (xy 266.7 60.96) (xy 270.51 60.96))
+    (stroke (width 0) (type default))
+  )
+  (wire (pts (xy 266.7 71.12) (xy 270.51 71.12))
+    (stroke (width 0) (type default))
+  )
+  (wire (pts (xy 266.7 66.04) (xy 270.51 66.04))
+    (stroke (width 0) (type default))
+  )
+  (wire (pts (xy 270.51 58.42) (xy 270.51 55.88))
+    (stroke (width 0) (type default))
+  )
+  (wire (pts (xy 270.51 60.96) (xy 270.51 63.5))
+    (stroke (width 0) (type default))
+  )
+  (wire (pts (xy 266.7 55.88) (xy 270.51 55.88))
+    (stroke (width 0) (type default))
+  )
+  (wire (pts (xy 270.51 66.04) (xy 270.51 68.58))
+    (stroke (width 0) (type default))
+  )
+  (wire (pts (xy 270.51 71.12) (xy 270.51 73.66))
+    (stroke (width 0) (type default))
+  )
+  (wire (pts (xy 266.7 76.2) (xy 270.51 76.2))
+    (stroke (width 0) (type default))
+  )
+  (wire (pts (xy 270.51 76.2) (xy 270.51 78.74))
+    (stroke (width 0) (type default))
+  )
+  (global_label "3.3V_ADCS" (shape output) (at 266.7 66.04 180) (fields_autoplaced)
+    (effects (font (size 1.27 1.27)) (justify right))
+    (property "Intersheetrefs" "${INTERSHEET_REFS}" (at 253.8761 66.04 0)
+      (effects (font (size 1.27 1.27)) (justify right) hide)
+    )
+  )
+  (global_label "3.3V_COMM" (shape output) (at 266.7 76.2 180) (fields_autoplaced)
+    (effects (font (size 1.27 1.27)) (justify right))
+    (property "Intersheetrefs" "${INTERSHEET_REFS}" (at 253.2109 76.2 0)
+      (effects (font (size 1.27 1.27)) (justify right) hide)
+    )
+  )
+  (global_label "5V_PAYLOAD" (shape output) (at 266.7 71.12 180) (fields_autoplaced)
+    (effects (font (size 1.27 1.27)) (justify right))
+    (property "Intersheetrefs" "${INTERSHEET_REFS}" (at 252.3641 71.12 0)
+      (effects (font (size 1.27 1.27)) (justify right) hide)
+    )
+  )
+  (global_label "+3.3V" (shape output) (at 266.7 55.88 180) (fields_autoplaced)
+    (effects (font (size 1.27 1.27)) (justify right))
+    (property "Intersheetrefs" "${INTERSHEET_REFS}" (at 258.1094 55.88 0)
+      (effects (font (size 1.27 1.27)) (justify right) hide)
+    )
+  )
+  (global_label "5V" (shape output) (at 266.7 60.96 180) (fields_autoplaced)
+    (effects (font (size 1.27 1.27)) (justify right))
+    (property "Intersheetrefs" "${INTERSHEET_REFS}" (at 261.4961 60.96 0)
+      (effects (font (size 1.27 1.27)) (justify right) hide)
+    )
+  )
+  (symbol (lib_id "PC104 conn:PTHF-126-02-GF-Q-368") (at 270.51 55.88 0) (unit 1)
     (in_bom yes) (on_board yes) (dnp no) (fields_autoplaced)
-    (property "Reference" "J1" (at 241.3 97.155 0)
+    (property "Reference" "J1" (at 284.48 98.425 0)
       (effects (font (size 1.524 1.524)) (justify left))
     )
-    (property "Value" "PTHF-126-02-GF-Q-368" (at 241.3 99.695 0)
+    (property "Value" "PTHF-126-02-GF-Q-368" (at 284.48 100.965 0)
       (effects (font (size 1.524 1.524)) (justify left))
     )
-    (property "Footprint" "CONN_PTHF-126-02-GF-Q-368_SAI" (at 227.33 54.61 0)
-      (effects (font (size 1.27 1.27) italic) hide)
-    )
-    (property "Datasheet" "PTHF-126-02-GF-Q-368" (at 227.33 54.61 0)
+    (property "Footprint" "CONN_PTHF-126-02-GF-Q-368_SAI" (at 270.51 55.88 0)
+      (effects (font (size 1.27 1.27) italic) hide)
+    )
+    (property "Datasheet" "PTHF-126-02-GF-Q-368" (at 270.51 55.88 0)
       (effects (font (size 1.27 1.27) italic) hide)
     )
@@
     )
   )
-  (symbol (lib_id "PC104 conn:PTHF-126-02-GF-Q-368") (at 125.73 55.88 0) (unit 2)
+  (symbol (lib_id "PC104 conn:PTHF-126-02-GF-Q-368") (at 133.35 95.25 90) (unit 2)
     (in_bom yes) (on_board yes) (dnp no) (fields_autoplaced)
-    (property "Reference" "J1" (at 139.7 98.425 0)
-      (effects (font (size 1.524 1.524)) (justify left))
-    )
-    (property "Value" "PTHF-126-02-GF-Q-368" (at 139.7 100.965 0)
-      (effects (font (size 1.524 1.524)) (justify left))
-    )
-    (property "Footprint" "CONN_PTHF-126-02-GF-Q-368_SAI" (at 125.73 55.88 0)
-      (effects (font (size 1.27 1.27) italic) hide)
-    )
-    (property "Datasheet" "PTHF-126-02-GF-Q-368" (at 125.73 55.88 0)
+    (property "Reference" "J1" (at 176.53 77.47 90)
+      (effects (font (size 1.524 1.524)))
+    )
+    (property "Value" "PTHF-126-02-GF-Q-368" (at 176.53 80.01 90)
+      (effects (font (size 1.524 1.524)))
+    )
+    (property "Footprint" "CONN_PTHF-126-02-GF-Q-368_SAI" (at 133.35 95.25 0)
+      (effects (font (size 1.27 1.27) italic) hide)
+    )
+    (property "Datasheet" "PTHF-126-02-GF-Q-368" (at 133.35 95.25 0)
       (effects (font (size 1.27 1.27) italic) hide)
     )
@@
     )
   )
-  (symbol (lib_id "PC104 conn:PTHF-126-02-GF-Q-368") (at 179.07 55.88 0) (unit 3)
+  (symbol (lib_id "PC104 conn:PTHF-126-02-GF-Q-368") (at 119.38 29.21 90) (unit 3)
     (in_bom yes) (on_board yes) (dnp no) (fields_autoplaced)
-    (property "Reference" "J1" (at 193.04 97.155 0)
-      (effects (font (size 1.524 1.524)) (justify left))
-    )
-    (property "Value" "PTHF-126-02-GF-Q-368" (at 193.04 99.695 0)
-      (effects (font (size 1.524 1.524)) (justify left))
-    )
-    (property "Footprint" "CONN_PTHF-126-02-GF-Q-368_SAI" (at 179.07 55.88 0)
-      (effects (font (size 1.27 1.27) italic) hide)
-    )
-    (property "Datasheet" "PTHF-126-02-GF-Q-368" (at 179.07 55.88 0)
-      (effects (font (size 1.27 1.27) italic) hide)
-    )
+    (property "Reference" "J1" (at 161.29 11.43 90)
+      (effects (font (size 1.524 1.524)))
+    )
+    (property "Value" "PTHF-126-02-GF-Q-368" (at 161.29 13.97 90)
+      (effects (font (size 1.524 1.524)))
+    )
+    (property "Footprint" "CONN_PTHF-126-02-GF-Q-368_SAI" (at 119.38 29.21 0)
+      (effects (font (size 1.27 1.27) italic) hide)
+    )
+    (property "Datasheet" "PTHF-126-02-GF-Q-368" (at 119.38 29.21 0)
+      (effects (font (size 1.27 1.27) italic) hide)
+    )

Commit message: updates
Connections:
- net +3.3V: now also J1.36, J1.37, J1.71, J1.72
- net 5V: now also J1.38, J1.39, J1.73, J1.74
- net 5V_COMM: now reaches J1.11
- net 5V_COMM: now also J1.12
- net USB_D-: now reaches J1.13
- net USB_D+: now reaches J1.14
- net BATTCH_EN: now reaches J1.16
- net SD_CARD_SPI2_MOSI: now reaches J1.19
- net SD_CARD_SPI2_MISO: now reaches J1.20
- net SD_CARD_SPI2_SCK: now reaches J1.21
- net SD_CARD_SPI2_NSS: now reaches J1.22
- net USART2_RX: now reaches J1.23
- net USART2_TX: now reaches J1.24
- net I2C2_SDA: now reaches J1.30
- net I2C2_SCL: now reaches J1.31
- net I2C3_SDA: now reaches J1.32
- net I2C3_SCL: now reaches J1.33
- net I2C1_SDA: now reaches J1.34
- net I2C1_SCL: now reaches J1.35
Other:
- moved on the sheet: J1B, J1C
